File: TesBoards/PA_HMC952/HMC952_TestBoard/HMC952_TestBoard.kicad_sch (KiCad schematic)
At the start: 27 parts

Commit message: changes
Parts:
- added J3: VDD, Connector_Molex:Molex_PicoBlade_53261-0271_1x02-1MP_P1.25mm_Horizontal, symbol GGS_Connectors:Picoblade_2x1_H
- added J4: VGG, Connector_Molex:Molex_PicoBlade_53261-0271_1x02-1MP_P1.25mm_Horizontal, symbol GGS_Connectors:Picoblade_2x1_H
- added J5: VDET, Connector_Molex:Molex_PicoBlade_53261-0271_1x02-1MP_P1.25mm_Horizontal, symbol GGS_Connectors:Picoblade_2x1_H
- SCRW1, SCRW2, SCRW3: renamed from SCRW?; footprint MountingHole:MountingHole_3.2mm_M3_Pad_Via -> MountingHole:MountingHole_2.7mm_M2.5_ISO14580
- gave numbers to parts that had none: 24
Connections:
- net RF_in is gone; now on net RF_In: J1.1 (RF)
- net Vg_PA2 is gone; now on net Vg_PA: C2.2, C5.2, C8.2, U1.7 (VGG2)
- net Vg_PA3 is gone; now on net Vg_PA: C3.2, C6.2, C9.2, U1.8 (VGG3)
- net GND: now also J3.2, J3.MP (MH2), J4.2, J4.MP (MH2), J5.2, J5.MP (MH2)
- net Vd_PA: now also J3.1
- net Vdet: now also J5.1
- net Vg_PA1 renamed Vg_PA
- net Vg_PA: now also J4.1
Other:
- note added: "Connectors"
- note added: "Heatsink"
- moved on the sheet: J1, J2, SCRW1, SCRW2, SCRW3, U1
