File: FrontEnd/HW/XCOMMS_RF/XCOMMS_RF.kicad_sch (KiCad schematic)
At the start: 60 parts, among them J1 SMP-MSLD-PCE-5T, J2 SMP-MSLD-PCE-5T, J3 SFC-110-T2-F-D-A-TR, U1 SIM-14+, U2 HMC788ALP2ETR, U3 HMC952ALP5GE, U5 HMC788ALP2ETR, U6 AD8031, U7 ADT7310

Commit message: XCOMMS RF Update
Parts:
- removed TP1, TP2, TP3, TP?: MS-156C3, GGS_Connectors:MS-156C3, symbol GGS_Connectors:MS-156C3
- added TP1, TP2, TP3, TP4: MS-156C, GGS_Connectors:CoaxialSwitch_Hirose_MS-156C3_Horizontal, symbol GGS_Connectors:MS-156C
- C12, C17, C20, C25, C28, C33, C36: footprint Capacitor_SMD:C_0805_2012Metric -> Capacitor_SMD:C_0603_1608Metric
- gave numbers to parts that had none: 5
Connections:
- net LO_EN is gone; now on net GND: J3.05
- net +3V3: now also J3.11; no longer J3.02
- net +5V: now also J3.03; no longer J3.01
- net AMP1_Out: no longer C1.1, L1.1, U2.5 (RFOUT)
- net AMP2_Out: now also C1.1, L1.1, U2.5 (RFOUT); no longer C22.1, L2.1, U5.5 (RFOUT)
- net FL_Out: now also TP2.C (In)
- net GND: now also J3.14, J3.16, J3.18, J3.20, TP1.G (GND), TP2.G (GND), TP3.G (GND), TP4.G (GND); no longer J3.06, J3.08, J3.11, J3.13
- net PA_RF_IN: now also TP3.A (Out)
- net PLL_CSB: now also J3.13; no longer J3.14
- net TP3_In: now also C1.2, TP3.C (In); no longer C22.2
- net Tx_LO: now also TP4.A (Out)
- net Tx_PM: now also J3.02; no longer J3.04
- net Vd_PA: now also J3.01; no longer J3.03
- net Vg_PA1: now also J3.08; no longer J3.20
- net Vg_PA2: now also J3.06; no longer J3.18
- net Vg_PA3: now also J3.04; no longer J3.16
- net AMP1_In renamed AMP2_In
- net AMP2_In: no longer U8.2 (RFIN)
- net RF_in renamed Mix_In
- net Mix_In: now also TP1.A (Out); no longer J2.1
- net TP1_Out renamed TP2_Out
- net TP2_Out: now also TP2.A (Out)
- net TP2_In renamed TP1_In
- net TP1_In: now also TP1.C (In); no longer C1.2
- new net AMP3_Out: C22.1, L2.1, U5.5 (RFOUT)
- new net RF_In: J2.1, U8.2 (RFIN)
- new net TP4_In: C22.2, TP4.C (In)
Other:
- sheet LocalOscillator ports: added none; removed LO_EN
- note added: "IC | V (V) | I (mA) | Power (mW) - - - - - - - - - - - - - - - - - - - PA | 5 | 1400 | ~2500 (class C) AMP1 | 4.5 | 65 | 290 AMP2 | 4.5 | 65 | 290 AMPLO | 4.5 | 65 | 290 PLL | 3.3 | 90 | 300 - - - - - - - - - - - - - - - - - - - Total | 3.7 W"
- note added: "Modifications: LO_EN eliminated -> PLL_CE"
- note added: "To do: Gruix Rogers R 0 Ohm"
- note removed: "IC | V (V) | I (mA) | Power (mW) - - - - - - - - - - - - - - - - - - - PA | 6 | 1400 | ~2500 (class C) AMP1 | 5 | 76 | 380 AMP2 | 5 | 56 | 280 HMC311LP3 AMPLO | 5 | 56 | 280 HMC311LP3 PLL | 3.3 | 90 | 300 - - - - - - - - - - - - - - - - - - - Total | 3.8 W"
- note removed: "To do: Amp 2.4 GHz Gruix Rogers R 0 Ohm"
- moved on the sheet: C2
