File: FrontEnd/HW/XCOMMS_RF/XCOMMS_RF.kicad_pcb (KiCad board)
At the start: 2 copper layers, 40 x 65 mm, 82 parts, among them J1 SMP-MSLD-PCE-5T, J2 SMP-MSLD-PCE-5T, J3 SFC-110-T2-F-D-A-TR, U1 SIM-14+, U2 HMC788ALP2ETR, U3 HMC952ALP5GE, U4 LMX2572RHAT, U5 HMC788ALP2ETR, U6 AD8031, U7 ADT7310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

Commit message: XCOMMS RF Update
Parts:
- added C52: 2.2uF, Capacitor_SMD:C_0603_1608Metric, F.Cu at (148.6, 84.4)
- added C53: 100pF, Capacitor_SMD:C_0402_1005Metric, F.Cu at (150.0, 84.7)
- added C54: 100pF, Capacitor_SMD:C_0402_1005Metric, F.Cu at (153.0, 87.1)
- added L3: 15nH, Inductor_SMD:L_0603_1608Metric, F.Cu at (152.2, 85.2)
- added TP4: MS-156C, GGS_Connectors:CoaxialSwitch_Hirose_MS-156C3_Horizontal, F.Cu at (165.1, 95.5)
- added U8: HMC788ALP2ETR, SamacSys_Footprints:SON65P200X200X90-7N-D, F.Cu at (153.0, 82.6)
- C12, C17, C20, C21, C25, C28, C33, C36, C6, C8, C9: footprint Capacitor_SMD:C_0805_2012Metric -> Capacitor_SMD:C_0603_1608Metric
- TP1, TP2, TP3: value MS-156C3 -> MS-156C; footprint GGS_Connectors:MS-156C3 -> GGS_Connectors:CoaxialSwitch_Hirose_MS-156C3_Horizontal
- moved TP3 35.0 mm to (152.4, 118.0), turned to -90 degrees
- moved TP2 13.4 mm to (152.4, 102.8)
- moved C47 11.5 mm to (169.8, 109.9), turned to -90 degrees
- moved R1 10.6 mm to (167.0, 101.4)
- moved C22 10.6 mm to (165.1, 98.3), turned to 90 degrees
- moved U5 10.6 mm to (165.1, 102.7)
- moved C41 10.5 mm to (160.6, 100.9)
- moved C42 10.5 mm to (162.1, 100.6)
- moved L2 10.5 mm to (164.3, 100.1)
- moved C30 10.5 mm to (167.0, 103.4)
- moved U1 10.4 mm to (159.1, 94.2)
- moved R3 10.3 mm to (169.2, 101.4)
- moved R4 10.3 mm to (170.4, 101.4)
- moved C29 10.2 mm to (165.2, 105.4)
- moved C44 10.1 mm to (169.2, 103.4)
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Connections:
- net /AMP1_In renamed /AMP2_In
- net /LocalOscillator/OSCINM renamed /LocalOscillator/VREGIN
- net /Mixer_Out renamed /Mix_Out
- C1 pad 1: /AMP1_Out -> /AMP2_Out
- C1 pad 2: /TP2_In -> /TP3_In
- C2 pad 1: /TP1_Out -> /TP2_Out
- C22 pad 1: /AMP2_Out -> /AMP3_Out
- C22 pad 2: /TP3_In -> /TP4_In
- J2 pad 1: /RF_in -> /RF_In
- J3 pad 01: +5V -> /Vd_PA
- J3 pad 02: +3V3 -> /Tx_PM
- J3 pad 03: /Vd_PA -> +5V
- J3 pad 04: /Tx_PM -> /Vg_PA3
- J3 pad 05: /LO_EN -> GND
- J3 pad 06: GND -> /Vg_PA2
- J3 pad 08: GND -> /Vg_PA1
- J3 pad 11: GND -> +3V3
- J3 pad 13: GND -> /PLL_CSB
- J3 pad 14: /PLL_CSB -> GND
- J3 pad 16: /Vg_PA3 -> GND
- J3 pad 18: /Vg_PA2 -> GND
- J3 pad 20: /Vg_PA1 -> GND
- L1 pad 1: /AMP1_Out -> /AMP2_Out
- L2 pad 1: /AMP2_Out -> /AMP3_Out
- U1 pad 2: /RF_in -> /Mix_In
- U2 pad 5: /AMP1_Out -> /AMP2_Out
- U5 pad 5: /AMP2_Out -> /AMP3_Out
- Y1 pad 1: /LO_EN -> /PLL_CE
Routing:
- net +3V3: track 153.3 -> 72.8 mm
- net GND: track 66.6 -> 27.1 mm, vias 190 -> 91
- net /LO_EN: track 30.7 -> 0.00 mm, vias 3 -> 0
- net +5V: track 66.0 -> 40.1 mm, vias 3 -> 4
- net /Vg_PA3: track 44.8 -> 27.2 mm, vias 3 -> 1
- net /Vg_PA2: track 44.4 -> 27.0 mm, vias 3 -> 1
- net /Vg_PA1: track 44.0 -> 27.0 mm, vias 3 -> 1
- net /SCK: track 81.6 -> 66.8 mm
- net /PLL_CE: track 27.7 -> 42.0 mm, vias 3 -> 4
- net /SDO: track 75.6 -> 62.2 mm
- net /PLL_CSB: track 37.9 -> 27.0 mm
- net /LocalOscillator/VREGIN: track 11.3 -> 2.16 mm
- net /LocalOscillator/OSCINP: track 10.9 -> 2.15 mm
- net /SDI: track 76.0 -> 67.6 mm, vias 3 -> 1
- net /RF_in: track 6.08 -> 0.00 mm
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
Commit message: XCOMMS Interface rebuild
Connections:
- C3 pad 2: +5V -> /Vd_AMP
- C4 pad 2: +5V -> /Vd_AMP
- C41 pad 2: +5V -> /Vd_AMP
- C42 pad 2: +5V -> /Vd_AMP
- C52 pad 2: +5V -> /Vd_AMP
- C53 pad 2: +5V -> /Vd_AMP
- J3 pad 03: +5V -> /Vd_AMP
- L1 pad 2: +5V -> /Vd_AMP
- L2 pad 2: +5V -> /Vd_AMP
- L3 pad 2: +5V -> /Vd_AMP
Routing:
- net +5V: track 40.1 -> 13.3 mm, vias 4 -> 1
- net /Vd_AMP: track 0.00 -> 24.8 mm, vias 0 -> 3
- net /RF_In: track 0.00 -> 1.99 mm
- net /AMP1_Out: track 0.00 -> 1.10 mm
- net /TP1_In: track 0.00 -> 0.97 mm

Commit message: XCOMMS RF
Parts:
- added REF**: Bike, GGS_Symbols:Bike, F.Cu at (140.0, 138.1)
- moved R10 41.2 mm to (143.4, 84.5), turned to -90 degrees
- moved R9 39.5 mm to (141.7, 84.5), turned to 90 degrees
- moved R5 39.2 mm to (140.1, 84.5), turned to -90 degrees
- moved U6 33.1 mm to (142.1, 88.1), turned to 180 degrees
- moved R8 27.2 mm to (143.3, 91.8), turned to 90 degrees
- moved R6 26.5 mm to (140.0, 91.8), turned to -90 degrees
- moved R7 25.1 mm to (141.6, 91.8), turned to -90 degrees
- moved C14 4.50 mm to (161.7, 104.6), turned to -90 degrees
- moved C13 2.50 mm to (160.0, 104.6), turned to -90 degrees
- moved C21 1.87 mm to (161.7, 116.2)
- moved C7 1.82 mm to (160.0, 116.2)
- moved C5 1.77 mm to (158.4, 116.2)
- moved C9 1.68 mm to (158.4, 104.6), turned to -90 degrees
- moved J3 1.17 mm to (140.5, 104.5)
- moved C41 0.58 mm to (160.0, 100.9)
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Connections:
- net /Vd_PA renamed /Vdd_PA
- C3 pad 2: /Vd_AMP -> /Vdd_AMP
- C4 pad 2: /Vd_AMP -> /Vdd_AMP
- C41 pad 2: /Vd_AMP -> /Vdd_AMP
- C42 pad 2: /Vd_AMP -> /Vdd_AMP
- C52 pad 2: /Vd_AMP -> /Vdd_AMP
- C53 pad 2: /Vd_AMP -> /Vdd_AMP
- J3 pad 02: /Tx_PM -> /Vg_PA3
- J3 pad 03: /Vd_AMP -> /Vdd_AMP
- J3 pad 04: /Vg_PA3 -> /Vg_PA2
- J3 pad 06: /Vg_PA2 -> /Vg_PA1
- J3 pad 08: /Vg_PA1 -> GND
- J3 pad 15: /SCK -> unconnected-(J3-Pad15)
- J3 pad 17: /SDO -> /SCK
- J3 pad 18: GND -> /Tx_PM
- J3 pad 19: /SDI -> /SDO
- J3 pad 20: GND -> /SDI
- L1 pad 2: /Vd_AMP -> /Vdd_AMP
- L2 pad 2: /Vd_AMP -> /Vdd_AMP
- L3 pad 2: /Vd_AMP -> /Vdd_AMP
- R5 pad 2: +5V -> /Vdd_AMP
- R6 pad 2: +5V -> /Vdd_AMP
- U6 pad 5: +5V -> /Vdd_AMP
Routing:
- net GND: track 27.1 -> 125.7 mm, vias 91 -> 445
- net /Vdd_AMP: track 0.00 -> 92.4 mm, vias 0 -> 5
- net +3V3: track 72.8 -> 121.2 mm, vias 8 -> 9
- net /Vref: track 16.7 -> 61.4 mm
- net /Vdet: track 27.4 -> 53.3 mm
- net /Vd_AMP: track 24.8 -> 0.00 mm, vias 3 -> 0
- net +5V: track 13.3 -> 0.00 mm, vias 1 -> 0
- net /LocalOscillator/VTune: track 26.4 -> 21.6 mm
- net /Tx_PM: track 11.6 -> 16.2 mm
- net /AMP2_Out: track 0.03 -> 3.47 mm
- net /Vdd_PA: track 67.9 -> 65.7 mm
- net /Vg_PA3: track 27.2 -> 25.2 mm
- net /PA_RF_IN: track 0.95 -> 2.89 mm
- net /FL_Out: track 0.00 -> 1.91 mm
- net /Vg_PA2: track 27.0 -> 25.3 mm
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Other:
- board text added: "ROGERS 4003C Layers = 2 Metalization = 35 um Thinkness = 0.508 mm (20 mils) Er = 3.55 tand = 0.0027"
- board text removed: "ROGERS 4350B Layers = 2 Metalization = 35 um Thinkness = 0.508 mm (20 mils) Er = 3.66 tand = 0.0037"
