File: TestBoards/PA_HMC952/HMC952_TestBoard/HMC952_TestBoard.kicad_sch (KiCad schematic)
At the start: 31 parts, among them J1 SMA, J2 SMA, J3 VDD, J4 VGG, J5 VDET, J6 VDET, U1 HMC952ALP5GE

Commit message: XCOMMS RF Update
Parts:
- removed J3: VDD, Connector_Molex:Molex_PicoBlade_53261-0271_1x02-1MP_P1.25mm_Horizontal, symbol GGS_Connectors:Picoblade_2x1_H
- removed J4: VGG, Connector_Molex:Molex_PicoBlade_53261-0271_1x02-1MP_P1.25mm_Horizontal, symbol GGS_Connectors:Picoblade_2x1_H
- removed J5, J6: VDET, Connector_Molex:Molex_PicoBlade_53261-0271_1x02-1MP_P1.25mm_Horizontal, symbol GGS_Connectors:Picoblade_2x1_H
- added J3, J4, J5: Conn_01x04, Connector_PinHeader_2.54mm:PinHeader_1x04_P2.54mm_Vertical, symbol Connector_Generic:Conn_01x04
Connections:
- net GND: now also J3.3 (Pin_3), J3.4 (Pin_4), J4.1 (Pin_1), J5.2 (Pin_2), J5.4 (Pin_4)
- net Vd_PA: now also J3.1 (Pin_1), J3.2 (Pin_2)
- net Vdet: now also J5.1 (Pin_1)
- net Vref: now also J5.3 (Pin_3)
- removed net Vg_PA: C1.2, C2.2, C3.2, C4.2, C5.2, C6.2, C7.2, C8.2, C9.2, U1.6 (VGG1), U1.7 (VGG2), U1.8 (VGG3)
- new net Vg_PA1: C1.2, C4.2, C7.2, J4.2 (Pin_2), U1.6 (VGG1)
- new net Vg_PA2: C2.2, C5.2, C8.2, J4.3 (Pin_3), U1.7 (VGG2)
- new net Vg_PA3: C3.2, C6.2, C9.2, J4.4 (Pin_4), U1.8 (VGG3)
Other:
- moved on the sheet: J1, J2
