File: FrontEnd/HW/XCOMMS_Interface/XCOMMS_Interface.kicad_pcb (KiCad board)
At the start: 4 copper layers, 40 x 65 mm, 113 parts, among them J1 TFC-110-02-F-D-A-P-FR, J2 PicoBlade01x05, J3 PicoBlade01x05, J4 PicoBlade01x02, U1 STM32L431KBUx, U10 MAX870EUK, U11 STM32L053R8Tx, U2 TPS56637, U3 TPS56637, U4 TPS56637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

Commit message: continuation of previous
Parts:
- moved TP7 0.22 mm to (133.4, 101.8)
- moved C38 0.22 mm to (138.8, 102.6)
- moved C39 0.22 mm to (143.8, 102.1)
- moved C40 0.22 mm to (140.5, 105.9)
- moved R20 0.22 mm to (136.5, 101.9)
- moved R21 0.22 mm to (136.5, 103.4)
- moved U10 0.22 mm to (141.3, 102.9)
Connections:
- U1 pad 10: unconnected-(U1-Pad10) -> /R_CSB
- U1 pad 19: unconnected-(U1-Pad19) -> /I2C1_SCL
- U1 pad 2: /RCC_IN -> unconnected-(U1-Pad2)
- U1 pad 20: unconnected-(U1-Pad20) -> /I2C1_SDA
- U1 pad 29: /I2C1_SCL -> unconnected-(U1-Pad29)
- U1 pad 3: /RCC_OUT -> unconnected-(U1-Pad3)
- U1 pad 30: /I2C1_SDA -> unconnected-(U1-Pad30)
- U1 pad 6: unconnected-(U1-Pad6) -> /RCC_IN_HSE
- U1 pad 9: /R_CSB -> unconnected-(U1-Pad9)
- U11 pad 17: /R_CSB -> unconnected-(U11-Pad17)
- U11 pad 20: unconnected-(U11-Pad20) -> /R_CSB
Routing:
- net +12V: track 109.4 -> 122.2 mm, vias 3 -> 5
- net +3V3: track 35.8 -> 27.5 mm, vias 1 -> 0
- net /NRST: track 7.73 -> 3.24 mm, vias 2 -> 1
- net /I2C1_SDA: track 10.5 -> 9.19 mm
- net /PLL_CSB: track 3.15 -> 1.84 mm

Commit message: XCOMMS RF
Parts:
- added C42: 100nF, Capacitor_SMD:C_0603_1608Metric, B.Cu at (145.4, 80.9)
- C41: value 7pF -> 100nF
- C6: value 7pF -> 1uF
- Y1: value ECS-.327-7-34QCS-TR -> TCXO_ECS; footprint Crystal:Crystal_SMD_3215-2Pin_3.2x1.5mm -> GGS_Miscellaneous:TCXO_ECS
- moved C3 17.7 mm to (147.8, 91.6), turned to 180 degrees
- moved C4 15.5 mm to (159.4, 77.7), turned to 0 degrees
- moved TP3 10.5 mm to (153.4, 110.7)
- moved TP2 8.43 mm to (133.2, 111.9)
- moved C13 7.22 mm to (162.8, 126.5), turned to 0 degrees
- moved J1 5.68 mm to (135.5, 104.5)
- moved C30 5.47 mm to (155.6, 93.9), turned to 180 degrees
- moved R22 4.36 mm to (163.2, 88.0), turned to 180 degrees
- moved C6 4.01 mm to (163.2, 84.7), turned to 180 degrees
- moved Y1 3.92 mm to (164.0, 87.1), turned to 180 degrees
- moved R1 3.80 mm to (159.4, 76.1), turned to 0 degrees
- moved C2 3.65 mm to (163.2, 91.8), turned to 0 degrees
- moved C23 3.47 mm to (140.5, 109.9), turned to 0 degrees
- moved D2 3.43 mm to (155.0, 110.3)
- moved D1 3.43 mm to (155.9, 111.8)
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Connections:
- net /5V_EN renamed /EN_5V
- net /6V_EN renamed /EN_6V
- C41 pad 1: /RCC_OUT -> +3V3
- C6 pad 1: /RCC_IN -> +3V3
- J1 pad 01: /Pout_PA -> /Vg_PA3
- J1 pad 03: /Vg_PA3 -> /Vg_PA2
- J1 pad 05: /Vg_PA2 -> /Vg_PA1
- J1 pad 07: /Vg_PA1 -> GND
- J1 pad 16: /SCK -> unconnected-(J1-Pad16)
- J1 pad 17: GND -> /Pout_PA
- J1 pad 18: /SDO -> /SCK
- J1 pad 19: GND -> /SDI
- J1 pad 20: /SDI -> /SDO
- U1 pad 22: /T_CSB -> unconnected-(U1-Pad22)
- U1 pad 26: unconnected-(U1-Pad26) -> /T_CSB
- U1 pad 27: /Tx_CE -> /PLL_CE
- U1 pad 6: /RCC_IN_HSE -> /RCC_IN
- U11 pad 45: /T_CSB -> unconnected-(U11-Pad45)
- U11 pad 55: unconnected-(U11-Pad55) -> /T_CSB
- U11 pad 56: /Tx_CE -> /PLL_CE
- U11 pad 6: /RCC_OUT -> unconnected-(U11-Pad6)
- Y1 pad 1: /RCC_IN -> +3V3
- Y1 pad 2: /RCC_OUT -> GND
Routing:
- net +12V: track 122.2 -> 33.0 mm, vias 5 -> 9
- net +3V3: track 27.5 -> 80.8 mm, vias 0 -> 13
- net /T_CSB: track 1.84 -> 54.0 mm, vias 0 -> 1
- net /PLL_CE: track 1.84 -> 52.9 mm, vias 0 -> 1
- net /SCK/SWCLK: track 3.24 -> 52.3 mm
- net /PLL_CSB: track 1.84 -> 49.9 mm
- net /EN_5V: track 2.15 -> 50.0 mm, vias 1 -> 2
- net /SCK: track 2.60 -> 50.2 mm, vias 1 -> 3
- net /TMS/SWDIO: track 3.27 -> 49.4 mm
- net /EN_6V: track 2.17 -> 41.2 mm, vias 1 -> 2
- net /SDI: track 2.64 -> 39.9 mm, vias 1 -> 3
- net /Vg_PA1: track 5.79 -> 42.9 mm
- net /NRST: track 3.24 -> 38.9 mm, vias 1 -> 3
- net /Pout_PA: track 4.31 -> 38.7 mm, vias 0 -> 2
- net +5V: track 18.0 -> 50.6 mm, vias 1 -> 3
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- added copper zone on B.Cu, net +12V
- added copper zone on In1.Cu, net +12V
- added copper zone on B.Cu, net +3V3
- added copper zone on In1.Cu, net +3V3
- added copper zone on B.Cu, net +5V
- added copper zone on In1.Cu, net /Vd_PA
- added copper zone on B.Cu, net /XCOMMS_PowerSupply/6V
Other:
- board text added: "JTAG"
- board text added: "OBC"
- board text added: "PWR"

Commit message: simplified PA gate control
Parts:
- removed C30, C31, C32: 1uF, Capacitor_SMD:C_0603_1608Metric
- removed C35, C36, C37, C38, C39, C40: 0.33uF, Capacitor_SMD:C_0603_1608Metric
- removed R13, R16, R20: 10k, Resistor_SMD:R_0603_1608Metric
- removed R14: 0R, Resistor_SMD:R_0603_1608Metric
- removed R15, R17, R18, R21: 20k, Resistor_SMD:R_0603_1608Metric
- removed R19: 5k, Resistor_SMD:R_0603_1608Metric
- removed TP5, TP6, TP7: TestPoint, TestPoint:TestPoint_Pad_D1.0mm
- removed U10, U9: MAX870EUK, Package_TO_SOT_SMD:SOT-23-5
- removed U5: TPS784, Package_TO_SOT_SMD:SOT-23-5
- removed U8: AD5160, Package_TO_SOT_SMD:SOT-23-8
- C29, C34: value 0.33uF -> 1uF
- moved C34 14.0 mm to (140.6, 105.1)
- moved TP4 13.9 mm to (135.6, 100.8), turned to 0 degrees
- moved U6 13.9 mm to (140.6, 102.0)
- moved C29 12.2 mm to (137.9, 100.1), turned to -90 degrees
- moved C33 11.8 mm to (140.6, 99.0), turned to 180 degrees
- moved R1 9.71 mm to (149.7, 77.1), turned to 90 degrees
- moved C3 9.03 mm to (138.8, 91.1), turned to 90 degrees
- moved C41 8.67 mm to (156.5, 80.9)
- moved C6 8.67 mm to (156.5, 79.2)
- moved C4 8.03 mm to (151.4, 77.1), turned to 90 degrees
- moved U1 7.03 mm to (146.9, 86.0)
- moved U11 7.03 mm to (146.9, 86.0)
- moved C5 6.96 mm to (156.5, 87.9)
- moved R22 6.96 mm to (156.5, 86.2)
- moved C42 6.91 mm to (138.9, 83.1)
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Connections:
- net /R_CSB renamed /V_PAControl
- net /XCOMMS_PowerSupply/Buck3V3_Comp renamed Net-(C27-Pad2)
- net /XCOMMS_PowerSupply/Vinv_in renamed /XCOMMS_PowerSupply/V_PAControl
- C29 pad 2: /XCOMMS_PowerSupply/Inv1_Out -> /Vg_PA
- J1 pad 01: /Vg_PA3 -> /Vg_PA
- J1 pad 03: /Vg_PA2 -> /Vg_PA
- J1 pad 05: /Vg_PA1 -> /Vg_PA
- TP4 pad 1: /Vg_PA1 -> /Vg_PA
- U6 pad 1: /XCOMMS_PowerSupply/Inv1_Out -> /Vg_PA
Routing:
- net GND: track 15.9 -> 77.7 mm, vias 99 -> 103
- net /Vg_PA1: track 42.9 -> 0.00 mm, vias 1 -> 0
- net /Vg_PA2: track 37.3 -> 0.00 mm, vias 1 -> 0
- net /Vg_PA3: track 31.5 -> 0.00 mm, vias 1 -> 0
- net /XCOMMS_PowerSupply/V_PAControl: track 29.2 -> 2.23 mm
- net /Vg_PA: track 0.00 -> 24.1 mm, vias 0 -> 1
- net /SDI: track 39.9 -> 20.2 mm, vias 3 -> 1
- net /SCK: track 50.2 -> 32.3 mm, vias 3 -> 1
- net +3V3: track 80.8 -> 63.5 mm, vias 13 -> 15
- net /V_PAControl: track 19.1 -> 3.65 mm
- net /XCOMMS_PowerSupply/LDO_Out: track 12.0 -> 0.00 mm, vias 2 -> 0
- net /SDO: track 33.6 -> 23.7 mm
- net /Pout_PA: track 38.7 -> 31.6 mm, vias 2 -> 1
- net /PLL_CSB: track 49.9 -> 43.2 mm
- net /PLL_CE: track 52.9 -> 46.5 mm
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- removed copper zone on B.Cu, net GND

Commit message: don't remember
Parts:
- added R13: 20k, Resistor_SMD:R_0603_1608Metric, B.Cu at (137.9, 103.1)
- added R14: 20k, Resistor_SMD:R_0603_1608Metric, B.Cu at (137.2, 105.4)
- moved Annotation1 57.0 mm to (157.2, 80.5)
- moved C33 0.70 mm to (140.6, 98.3)
- moved C34 0.58 mm to (140.6, 105.7)
- moved C29 0.07 mm to (137.9, 100.1)
Connections:
- C29 pad 2: /Vg_PA -> /XCOMMS_PowerSupply/InvOut
- TP4 pad 1: /Vg_PA -> /XCOMMS_PowerSupply/InvOut
- U6 pad 1: /Vg_PA -> /XCOMMS_PowerSupply/InvOut
Routing:
- net /Vg_PA: track 24.1 -> 17.0 mm
- net /XCOMMS_PowerSupply/InvOut: track 0.00 -> 5.81 mm
- net GND: track 77.7 -> 78.9 mm, vias 103 -> 104
- net /XCOMMS_PowerSupply/Inv_C-: track 4.89 -> 5.72 mm
- net /XCOMMS_PowerSupply/V_PAControl: track 2.23 -> 2.94 mm
- net /XCOMMS_PowerSupply/Inv_C+: track 2.05 -> 2.63 mm
Other:
- board text added: "8"

Commit message: IDK
Parts:
- moved C33 0.40 mm to (140.6, 98.7)
- moved C34 0.26 mm to (140.6, 105.4)
Routing:
- net /XCOMMS_PowerSupply/6V: track 12.5 -> 15.2 mm
- net GND: track 78.9 -> 78.3 mm
- net /XCOMMS_PowerSupply/Inv_C-: track 5.72 -> 5.20 mm
Other:
- board text added: "v2.2"
- board text removed: "v2"
