File: FrontEnd/HW/XCOMMS_Interface/XCOMMS_PowerSupply.kicad_sch (KiCad schematic)
At the start: 50 parts, among them U2 TPS56637, U3 TPS56637, U4 TPS56637, U6 MAX870EUK, U7 INA290

Commit message: don't remember
Parts:
- added R13, R14: 20k, Resistor_SMD:R_0603_1608Metric, symbol Device:R
Connections:
- net GND: now also R14.1
- net Vg_PA: now also R13.2, R14.2; no longer C29.2, TP4.1, U6.1 (OUT)
- new net InvOut: C29.2, R13.1, TP4.1, U6.1 (OUT)
Changed lines of the file:
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@@
   (junction (at 119.38 50.8) (diameter 0) (color 0 0 0 0)
+  )
+  (junction (at 251.46 39.37) (diameter 0) (color 0 0 0 0)
   )
   (junction (at 57.15 99.06) (diameter 0) (color 0 0 0 0)
@@
     (stroke (width 0) (type default) (color 0 0 0 0))
   )
+  (wire (pts (xy 229.87 39.37) (xy 240.03 39.37))
+    (stroke (width 0) (type default) (color 0 0 0 0))
+  )
   (wire (pts (xy 128.27 105.41) (xy 129.54 105.41))
     (stroke (width 0) (type default) (color 0 0 0 0))
@@
     (stroke (width 0) (type default) (color 0 0 0 0))
   )
+  (wire (pts (xy 251.46 39.37) (xy 255.27 39.37))
+    (stroke (width 0) (type default) (color 0 0 0 0))
+  )
   (wire (pts (xy 114.3 50.8) (xy 119.38 50.8))
     (stroke (width 0) (type default) (color 0 0 0 0))
@@
     (stroke (width 0) (type default) (color 0 0 0 0))
   )
+  (wire (pts (xy 251.46 53.34) (xy 251.46 49.53))
+    (stroke (width 0) (type default) (color 0 0 0 0))
+  )
   (wire (pts (xy 81.28 63.5) (xy 49.53 63.5))
     (stroke (width 0) (type default) (color 0 0 0 0))
@@
     (stroke (width 0) (type default) (color 0 0 0 0))
   )
+  (wire (pts (xy 251.46 39.37) (xy 247.65 39.37))
+    (stroke (width 0) (type default) (color 0 0 0 0))
+  )
   (wire (pts (xy 119.38 105.41) (xy 119.38 104.14))
     (stroke (width 0) (type default) (color 0 0 0 0))
@@
     (stroke (width 0) (type default) (color 0 0 0 0))
   )
+  (wire (pts (xy 251.46 39.37) (xy 251.46 41.91))
+    (stroke (width 0) (type default) (color 0 0 0 0))
+  )
   (wire (pts (xy 85.09 52.07) (xy 85.09 50.8))
     (stroke (width 0) (type default) (color 0 0 0 0))
@@
     (stroke (width 0) (type default) (color 0 0 0 0))
   )
-  (wire (pts (xy 241.3 39.37) (xy 229.87 39.37))
-    (stroke (width 0) (type default) (color 0 0 0 0))
-  )
   (wire (pts (xy 193.04 96.52) (xy 187.96 96.52))
     (stroke (width 0) (type default) (color 0 0 0 0))
@@
     (effects (font (size 1.27 1.27)) (justify left bottom))
   )
+  (label "InvOut" (at 219.71 39.37 0)
+    (effects (font (size 1.27 1.27)) (justify left bottom))
+  )
   (label "Buck5V_SW" (at 95.25 86.36 0)
     (effects (font (size 1.27 1.27)) (justify left bottom))
@@
     (effects (font (size 1.27 1.27)) (justify left bottom))
   )
-  (hierarchical_label "Vg_PA" (shape input) (at 241.3 39.37 0)
+  (hierarchical_label "Vg_PA" (shape input) (at 255.27 39.37 0)
     (effects (font (size 1.27 1.27)) (justify left))
   )
@@
     )
     (pin "1")
+  )
+  (symbol (lib_id "Device:R") (at 251.46 45.72 180) (unit 1)
+    (in_bom yes) (on_board yes) (fields_autoplaced)
+    (property "Reference" "R14" (id 0) (at 254 44.4499 0)
+      (effects (font (size 1.27 1.27)) (justify right))
+    )
+    (property "Value" "20k" (id 1) (at 254 46.9899 0)
+      (effects (font (size 1.27 1.27)) (justify right))
+    )
+    (property "Footprint" "Resistor_SMD:R_0603_1608Metric" (id 2) (at 253.238 45.72 90)
+      (effects (font (size 1.27 1.27)) hide)
+    )
+    (property "Datasheet" "~" (id 3) (at 251.46 45.72 0)
+      (effects (font (size 1.27 1.27)) hide)
+    )
+    (pin "1")
+    (pin "2")
   )
   (symbol (lib_id "power:+12V") (at 44.45 153.67 0) (unit 1)
@@
     (pin "1")
   )
+  (symbol (lib_id "Device:R") (at 243.84 39.37 90) (unit 1)
+    (in_bom yes) (on_board yes) (fields_autoplaced)
+    (property "Reference" "R13" (id 0) (at 243.84 33.02 90))
+    (property "Value" "20k" (id 1) (at 243.84 35.56 90))
+    (property "Footprint" "Resistor_SMD:R_0603_1608Metric" (id 2) (at 243.84 41.148 90)
+      (effects (font (size 1.27 1.27)) hide)
+    )
+    (property "Datasheet" "~" (id 3) (at 243.84 39.37 0)
+      (effects (font (size 1.27 1.27)) hide)
+    )
+    (pin "1")
+    (pin "2")
+  )
   (symbol (lib_id "power:GND") (at 149.86 52.07 0) (unit 1)
     (in_bom yes) (on_board yes) (fields_autoplaced)
@@
     (pin "2")
   )
+  (symbol (lib_id "power:GND") (at 251.46 53.34 0) (unit 1)
+    (in_bom yes) (on_board yes) (fields_autoplaced)
+    (property "Reference" "#PWR04" (id 0) (at 251.46 59.69 0)
+      (effects (font (size 1.27 1.27)) hide)
+    )
+    (property "Value" "GND" (id 1) (at 251.46 58.42 0))
+    (property "Footprint" "" (id 2) (at 251.46 53.34 0)
+      (effects (font (size 1.27 1.27)) hide)
+    )
+    (property "Datasheet" "" (id 3) (at 251.46 53.34 0)
+      (effects (font (size 1.27 1.27)) hide)
+    )
+    (pin "1")
+  )
   (symbol (lib_id "Device:R") (at 119.38 165.1 0) (unit 1)

Commit message: IDK
Other:
- moved on the sheet: C28, C29, C33, C34, R13, R14, Rsense1, Rsense2, TP4, U6, U7
