File: FrontEnd/HW/XCOMMS_EGSE/XCOMMS_EGSE/XCOMMS_EGSE.kicad_pcb (KiCad board)
At the start: 2 copper layers, 170 x 80 mm, 12 parts, among them J1 TFC-110-02-F-D-A-P-FR, J2 Conn_01x10, J3 Conn_01x10, J5 TFC-110-02-F-D-A-P-FR

Commit message: IDK
Parts:
- added REF**: Prj, GGS_Symbols:Prj, F.Cu at (60.0, 55.0)
- added REF**: GGS, GGS_Symbols:GGS, F.Cu at (85.0, 55.5)
- added REF**: NSL, GGS_Symbols:NSL, F.Cu at (142.7, 60.9)
- added REF**: UPC, GGS_Symbols:UPC, F.Cu at (128.0, 59.0)
- moved H5 76.0 mm to (104.0, 62.0)
- moved H6 76.0 mm to (104.0, 121.0)
- moved H7 76.0 mm to (138.0, 62.0)
- moved H8 76.0 mm to (138.0, 121.0)
- moved J5 76.0 mm to (108.5, 91.5)
- moved H3 71.9 mm to (62.0, 121.0), turned to 180 degrees
- moved H4 68.5 mm to (62.0, 62.0), turned to 180 degrees
- moved H1 68.0 mm to (96.0, 121.0), turned to 180 degrees
- moved H2 64.4 mm to (96.0, 62.0), turned to 180 degrees
- moved J2 34.2 mm to (146.0, 88.3), turned to 180 degrees
- moved J1 21.1 mm to (91.5, 91.5), turned to 90 degrees
- moved J3 7.21 mm to (146.0, 94.1)
Routing:
- net Net-(J1-Pad14): track 0.00 -> 95.4 mm, vias 0 -> 2
- net Net-(J1-Pad10): track 54.0 -> 99.0 mm, vias 0 -> 2
- net Net-(J1-Pad06): track 55.1 -> 99.3 mm, vias 0 -> 2
- net Net-(J1-Pad04): track 55.6 -> 99.8 mm, vias 0 -> 2
- net Net-(J1-Pad02): track 56.1 -> 99.5 mm, vias 0 -> 2
- net Net-(J1-Pad18): track 52.5 -> 94.7 mm, vias 0 -> 2
- net Net-(J1-Pad20): track 52.0 -> 94.0 mm, vias 0 -> 2
- net Net-(J1-Pad12): track 53.5 -> 95.4 mm, vias 0 -> 2
- net Net-(J1-Pad16): track 53.0 -> 94.9 mm, vias 0 -> 2
- net Net-(J1-Pad01): track 109.7 -> 68.6 mm, vias 0 -> 2
- net Net-(J1-Pad03): track 104.8 -> 68.1 mm, vias 0 -> 2
- net Net-(J1-Pad05): track 100.0 -> 69.2 mm, vias 0 -> 2
- net Net-(J1-Pad07): track 92.6 -> 69.4 mm, vias 0 -> 2
- net Net-(J1-Pad09): track 86.4 -> 70.8 mm, vias 0 -> 2
- net Net-(J1-Pad19): track 59.7 -> 75.0 mm, vias 0 -> 2
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Other:
- board size 170 x 80 mm -> 100 x 80 mm
- board text added: "19 17 15 13 11 9 7 5 3 1"
- board text added: "20 18 16 14 12 10 8 6 4 2"
- board text added: "8"
